File: hardware/Display Adapter/Display Adapter.kicad_sch (KiCad schematic)
At the start: 2 parts, among them J1 IDC-Header_2x07_P2.54mm, J2 ILI9341 2.8" touch TFT

Commit message: Update Display Adapter project to Kicad 7.0.2
Parts:
- J2: symbol Connector:Conn_01x14_Male -> Connector:Conn_01x14_Pin; now in the parts list
