File: hardware/Control Board/IoT12 Control Board.kicad_sch (KiCad schematic)
At the start: 4 parts

Commit message: Start of next iteration.
Parts:
- H1, H2, H3, H4: symbol Mechanical:MountingHole -> Mechanical:MountingHole_Pad; now left out of the parts list
Connections:
- no-connect marks 0 -> 4
Other:
- company: (none) -> https://github.com/atoomnetmarc/IoT12
- title: IoT12-hardware -> IoT12 Control Board
